File: pcb/combinador/combinador.kicad_sch (KiCad schematic)
At the start: 17 parts, among them J1 SMA, J2 SMA, J3 SMA, J4 SMA, J5 SMA, J6 SMA, U1 1.7GHz, U2 2.5GHz, U3 3.5GHz, U4 4.1GHz

Commit message: Actualización
Agregado de modelo 3d de conectores, correxión en la medida de los pads de los resistores. Agregado de etiquetas de cada acoplador.
Parts:
- J1, J2, J3, J4, J5, J6: footprint footprint_project_library:SMA -> footprint_project_library:SMA_horizontal_microstrip
- R1, R2, R3, R4, R5, R6, R7: footprint Resistor_SMD:R_0603_1608Metric -> footprint_project_library:R_0603
Changed lines of the file:
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@@
       (effects (font (size 1.27 1.27)) (justify left))
     )
-    (property "Footprint" "footprint_project_library:SMA" (at 214.63 91.44 0)
+    (property "Footprint" "footprint_project_library:SMA_horizontal_microstrip" (at 214.63 91.44 0)
       (effects (font (size 1.27 1.27)) hide)
     )
@@
       (effects (font (size 1.27 1.27)) (justify left))
     )
-    (property "Footprint" "Resistor_SMD:R_0603_1608Metric" (at 111.506 115.824 90)
+    (property "Footprint" "footprint_project_library:R_0603" (at 111.506 115.824 90)
       (effects (font (size 1.27 1.27)) hide)
     )
@@
       (effects (font (size 1.27 1.27)) (justify left))
     )
-    (property "Footprint" "Resistor_SMD:R_0603_1608Metric" (at 138.176 115.824 90)
+    (property "Footprint" "footprint_project_library:R_0603" (at 138.176 115.824 90)
       (effects (font (size 1.27 1.27)) hide)
     )
@@
       (effects (font (size 1.27 1.27)) (justify left))
     )
-    (property "Footprint" "Resistor_SMD:R_0603_1608Metric" (at 75.946 98.044 90)
+    (property "Footprint" "footprint_project_library:R_0603" (at 75.946 98.044 90)
       (effects (font (size 1.27 1.27)) hide)
     )
@@
       (effects (font (size 1.27 1.27)) (justify left))
     )
-    (property "Footprint" "footprint_project_library:SMA" (at 173.99 111.76 0)
+    (property "Footprint" "footprint_project_library:SMA_horizontal_microstrip" (at 173.99 111.76 0)
       (effects (font (size 1.27 1.27)) hide)
     )
@@
       (effects (font (size 1.27 1.27)) (justify left))
     )
-    (property "Footprint" "Resistor_SMD:R_0603_1608Metric" (at 164.846 115.824 90)
+    (property "Footprint" "footprint_project_library:R_0603" (at 164.846 115.824 90)
       (effects (font (size 1.27 1.27)) hide)
     )
@@
       (effects (font (size 1.27 1.27)) (justify left))
     )
-    (property "Footprint" "Resistor_SMD:R_0603_1608Metric" (at 94.996 98.044 90)
+    (property "Footprint" "footprint_project_library:R_0603" (at 94.996 98.044 90)
       (effects (font (size 1.27 1.27)) hide)
     )
@@
       (effects (font (size 1.27 1.27)) (justify left))
     )
-    (property "Footprint" "footprint_project_library:SMA" (at 147.32 111.76 0)
+    (property "Footprint" "footprint_project_library:SMA_horizontal_microstrip" (at 147.32 111.76 0)
       (effects (font (size 1.27 1.27)) hide)
     )
@@
       (effects (font (size 1.27 1.27)) (justify left))
     )
-    (property "Footprint" "Resistor_SMD:R_0603_1608Metric" (at 85.344 90.424 90)
+    (property "Footprint" "footprint_project_library:R_0603" (at 85.344 90.424 90)
       (effects (font (size 1.27 1.27)) hide)
     )
@@
       (effects (font (size 1.27 1.27)) (justify left))
     )
-    (property "Footprint" "footprint_project_library:SMA" (at 120.65 111.76 0)
+    (property "Footprint" "footprint_project_library:SMA_horizontal_microstrip" (at 120.65 111.76 0)
       (effects (font (size 1.27 1.27)) hide)
     )
@@
       (effects (font (size 1.27 1.27)) (justify left))
     )
-    (property "Footprint" "footprint_project_library:SMA" (at 60.96 91.44 0)
+    (property "Footprint" "footprint_project_library:SMA_horizontal_microstrip" (at 60.96 91.44 0)
       (effects (font (size 1.27 1.27)) hide)
     )
@@
       (effects (font (size 1.27 1.27)) (justify left))
     )
-    (property "Footprint" "Resistor_SMD:R_0603_1608Metric" (at 191.516 115.824 90)
+    (property "Footprint" "footprint_project_library:R_0603" (at 191.516 115.824 90)
       (effects (font (size 1.27 1.27)) hide)
     )
@@
       (effects (font (size 1.27 1.27)) (justify left))
     )
-    (property "Footprint" "footprint_project_library:SMA" (at 200.66 111.76 0)
-      (effects (font (size 1.27 1.27)) hide)
-    )
+    (property "Footprint" "footprint_project_library:SMA_horizontal_microstrip" (at 200.66 111.76 0)
+      (effects (font (size 1.27 1.27)) hide)
+    )
